File: hardware/schematics/car/car.kicad_sch (KiCad schematic)
At the start: 21 parts, among them M1 Motor_Servo, Q1 PMOS, SW1 SW_SPST, SW2 SW_Push, SW3 SW_Push, U1 VL53L0CXV0DH1, U10 Mini-560, U11 JGA25-37x, U2 VL53L0CXV0DH1, U3 VL53L0CXV0DH1, U4 Pixy2, U6 TB6612FNG, U7 SparkFun OTOS, U8 SWD debug probe, U9 Mini-360

Commit message: [Schematic] Fix footprints.
Parts:
- U1, U2, U3: footprint xlnc-foot:VL53L0/1XV2_PinHeader_1x06_P2.54mm_Vertical -> xlnc-foot:VL53L0_1XV2_PinHeader_1x06_P2.54mm_Vertical
Changed lines of the file:
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@@
 			)
 		)
-		(property "Footprint" "xlnc-foot:VL53L0/1XV2_PinHeader_1x06_P2.54mm_Vertical"
+		(property "Footprint" "xlnc-foot:VL53L0_1XV2_PinHeader_1x06_P2.54mm_Vertical"
 			(at 47.625 86.36 0)
 			(hide yes)
@@
 			)
 		)
-		(property "Footprint" "xlnc-foot:VL53L0/1XV2_PinHeader_1x06_P2.54mm_Vertical"
+		(property "Footprint" "xlnc-foot:VL53L0_1XV2_PinHeader_1x06_P2.54mm_Vertical"
 			(at 47.625 46.99 0)
 			(hide yes)
@@
 			)
 		)
-		(property "Footprint" "xlnc-foot:VL53L0/1XV2_PinHeader_1x06_P2.54mm_Vertical"
+		(property "Footprint" "xlnc-foot:VL53L0_1XV2_PinHeader_1x06_P2.54mm_Vertical"
 			(at 50.165 135.89 0)
 			(hide yes)
